Commit message: fix: base_linkの原点を修正

File: rcj2025_description/urdf/rcj2025.xacro (robot description, xacro)
@@ -6,5 +6,5 @@
 <link name="base_link">
   <inertial>
-    <origin xyz="-0.0008436056640299374 0.08187967201339755 -0.0021723659327403414" rpy="0 0 0"/>
+    <origin xyz="-0.0008436056640299374 0.07287967201339762 -0.002172365932740341" rpy="0 0 0"/>
     <mass value="6.211712403129365"/>
     <inertia ixx="0.020157" iyy="0.025166" izz="0.014889" ixy="0.00016" iyz="-0.000113" ixz="5.6e-05"/>
@@ -26,10 +26,10 @@
 <link name="wheel_left_forward_link_1">
   <inertial>
-    <origin xyz="0.0038321243790345877 -0.009000829458104417 0.0003539119469893326" rpy="0 0 0"/>
+    <origin xyz="0.0038321243790345877 -8.294581043746807e-07 0.0003539119469892979" rpy="0 0 0"/>
     <mass value="0.30797982883853386"/>
     <inertia ixx="0.000267" iyy="0.000139" izz="0.000139" ixy="0.0" iyz="0.0" ixz="0.0"/>
   </inertial>
   <visual>
-    <origin xyz="-0.074905 -0.050003 -0.044995" rpy="0 0 0"/>
+    <origin xyz="-0.074905 -0.032003 -0.044995" rpy="0 0 0"/>
     <geometry>
       <mesh filename="file://$(find rcj2025_description)/meshes/wheel_left_forward_link_1.stl" scale="0.001 0.001 0.001"/>
@@ -38,5 +38,5 @@
   </visual>
   <collision>
-    <origin xyz="-0.074905 -0.050003 -0.044995" rpy="0 0 0"/>
+    <origin xyz="-0.074905 -0.032003 -0.044995" rpy="0 0 0"/>
     <geometry>
       <mesh filename="file://$(find rcj2025_description)/meshes/wheel_left_forward_link_1.stl" scale="0.001 0.001 0.001"/>
@@ -46,10 +46,10 @@
 <link name="wheel_right_forward_link_1">
   <inertial>
-    <origin xyz="-0.0038321243830769514 -0.009003458642732436 0.00034373391199247344" rpy="0 0 0"/>
+    <origin xyz="-0.0038321243830769514 -3.458642732385997e-06 0.0003437339119924457" rpy="0 0 0"/>
     <mass value="0.30797982860031553"/>
     <inertia ixx="0.000267" iyy="0.000139" izz="0.000139" ixy="-0.0" iyz="-0.0" ixz="-0.0"/>
   </inertial>
   <visual>
-    <origin xyz="0.074905 -0.050003 -0.044995" rpy="0 0 0"/>
+    <origin xyz="0.074905 -0.032003 -0.044995" rpy="0 0 0"/>
     <geometry>
       <mesh filename="file://$(find rcj2025_description)/meshes/wheel_right_forward_link_1.stl" scale="0.001 0.001 0.001"/>
@@ -58,5 +58,5 @@
   </visual>
   <collision>
-    <origin xyz="0.074905 -0.050003 -0.044995" rpy="0 0 0"/>
+    <origin xyz="0.074905 -0.032003 -0.044995" rpy="0 0 0"/>
     <geometry>
       <mesh filename="file://$(find rcj2025_description)/meshes/wheel_right_forward_link_1.stl" scale="0.001 0.001 0.001"/>
@@ -66,10 +66,10 @@
 <link name="wheel_right_backward_link_1">
   <inertial>
-    <origin xyz="-0.0038321243783342313 -0.00899395860298674 -0.00012307261745360398" rpy="0 0 0"/>
+    <origin xyz="-0.0038321243783342313 6.041397013302474e-06 -0.00012307261745363868" rpy="0 0 0"/>
     <mass value="0.3079798288624377"/>
     <inertia ixx="0.000267" iyy="0.000139" izz="0.000139" ixy="-0.0" iyz="-0.0" ixz="0.0"/>
   </inertial>
   <visual>
-    <origin xyz="0.074905 -0.050003 0.044995" rpy="0 0 0"/>
+    <origin xyz="0.074905 -0.032003 0.044995" rpy="0 0 0"/>
     <geometry>
       <mesh filename="file://$(find rcj2025_description)/meshes/wheel_right_backward_link_1.stl" scale="0.001 0.001 0.001"/>
@@ -78,5 +78,5 @@
   </visual>
   <collision>
-    <origin xyz="0.074905 -0.050003 0.044995" rpy="0 0 0"/>
+    <origin xyz="0.074905 -0.032003 0.044995" rpy="0 0 0"/>
     <geometry>
       <mesh filename="file://$(find rcj2025_description)/meshes/wheel_right_backward_link_1.stl" scale="0.001 0.001 0.001"/>
@@ -86,10 +86,10 @@
 <link name="wheel_left_backward_link_1">
   <inertial>
-    <origin xyz="0.003832124382646254 -0.009003945927425837 -0.0003437082381777534" rpy="0 0 0"/>
+    <origin xyz="0.003832124382646254 -3.945927425814955e-06 -0.0003437082381777881" rpy="0 0 0"/>
     <mass value="0.30797982861500756"/>
     <inertia ixx="0.000267" iyy="0.000139" izz="0.000139" ixy="0.0" iyz="0.0" ixz="-0.0"/>
   </inertial>
   <visual>
-    <origin xyz="-0.074905 -0.050003 0.044995" rpy="0 0 0"/>
+    <origin xyz="-0.074905 -0.032003 0.044995" rpy="0 0 0"/>
     <geometry>
       <mesh filename="file://$(find rcj2025_description)/meshes/wheel_left_backward_link_1.stl" scale="0.001 0.001 0.001"/>
@@ -98,5 +98,5 @@
   </visual>
   <collision>
-    <origin xyz="-0.074905 -0.050003 0.044995" rpy="0 0 0"/>
+    <origin xyz="-0.074905 -0.032003 0.044995" rpy="0 0 0"/>
     <geometry>
       <mesh filename="file://$(find rcj2025_description)/meshes/wheel_left_backward_link_1.stl" scale="0.001 0.001 0.001"/>
@@ -105,5 +105,5 @@
 </link>
 <joint name="回転 100" type="continuous">
-  <origin xyz="0.074905 0.050003 0.044995" rpy="0 0 0"/>
+  <origin xyz="0.074905 0.032003 0.044995" rpy="0 0 0"/>
   <parent link="base_link"/>
   <child link="wheel_left_forward_link_1"/>
@@ -111,5 +111,5 @@
 </joint>
 <joint name="回転 101" type="continuous">
-  <origin xyz="-0.074905 0.050003 0.044995" rpy="0 0 0"/>
+  <origin xyz="-0.074905 0.032003 0.044995" rpy="0 0 0"/>
   <parent link="base_link"/>
   <child link="wheel_right_forward_link_1"/>
@@ -117,5 +117,5 @@
 </joint>
 <joint name="回転 102" type="continuous">
-  <origin xyz="-0.074905 0.050003 -0.044995" rpy="0 0 0"/>
+  <origin xyz="-0.074905 0.032003 -0.044995" rpy="0 0 0"/>
   <parent link="base_link"/>
   <child link="wheel_right_backward_link_1"/>
@@ -123,5 +123,5 @@
 </joint>
 <joint name="回転 103" type="continuous">
-  <origin xyz="0.074905 0.050003 -0.044995" rpy="0 0 0"/>
+  <origin xyz="0.074905 0.032003 -0.044995" rpy="0 0 0"/>
   <parent link="base_link"/>
   <child link="wheel_left_backward_link_1"/>

Commit message: feat: spawn gazebo sim

File: rcj2025_description/urdf/rcj2025.xacro (robot description, xacro)
@@ -4,4 +4,10 @@
 <xacro:include filename="$(find rcj2025_description)/urdf/rcj2025.trans" />
 <xacro:include filename="$(find rcj2025_description)/urdf/rcj2025.gazebo" />
+<link name="base_footprint"/>
+<joint name="base_link_joint" type="fixed">
+  <origin xyz="0 0.009 0" rpy="0 0 0"/>
+  <parent link="base_footprint"/>
+  <child link="base_link"/>
+</joint>
 <link name="base_link">
   <inertial>

Commit message: feat: /cmd_velで動いた

File: rcj2025_description/urdf/rcj2025.xacro (robot description, xacro)
@@ -4,10 +4,4 @@
 <xacro:include filename="$(find rcj2025_description)/urdf/rcj2025.trans" />
 <xacro:include filename="$(find rcj2025_description)/urdf/rcj2025.gazebo" />
-<link name="base_footprint"/>
-<joint name="base_link_joint" type="fixed">
-  <origin xyz="0 0.009 0" rpy="0 0 0"/>
-  <parent link="base_footprint"/>
-  <child link="base_link"/>
-</joint>
 <link name="base_link">
   <inertial>
@@ -110,5 +104,5 @@
   </collision>
 </link>
-<joint name="回転 100" type="continuous">
+<joint name="wheel_left_forward_joint" type="continuous">
   <origin xyz="0.074905 0.032003 0.044995" rpy="0 0 0"/>
   <parent link="base_link"/>
@@ -116,5 +110,5 @@
   <axis xyz="1.0 -0.0 -0.0"/>
 </joint>
-<joint name="回転 101" type="continuous">
+<joint name="wheel_right_forward_joint" type="continuous">
   <origin xyz="-0.074905 0.032003 0.044995" rpy="0 0 0"/>
   <parent link="base_link"/>
@@ -122,5 +116,5 @@
   <axis xyz="1.0 0.0 0.0"/>
 </joint>
-<joint name="回転 102" type="continuous">
+<joint name="wheel_right_backward_joint" type="continuous">
   <origin xyz="-0.074905 0.032003 -0.044995" rpy="0 0 0"/>
   <parent link="base_link"/>
@@ -128,5 +122,5 @@
   <axis xyz="-1.0 -0.0 0.0"/>
 </joint>
-<joint name="回転 103" type="continuous">
+<joint name="wheel_left_backward_joint" type="continuous">
   <origin xyz="0.074905 0.032003 -0.044995" rpy="0 0 0"/>
   <parent link="base_link"/>

Commit message: fix: モデルの座標系をgazeboに合わせるように修正

File: rcj2025_description/urdf/rcj2025.xacro (robot description, xacro)
@@ -6,7 +6,7 @@
 <link name="base_link">
   <inertial>
-    <origin xyz="-0.0008436056640299374 0.07287967201339762 -0.002172365932740341" rpy="0 0 0"/>
+    <origin xyz="-0.002172365932740349 -0.0008436056640299366 0.07287967201339762" rpy="0 0 0"/>
     <mass value="6.211712403129365"/>
-    <inertia ixx="0.020157" iyy="0.025166" izz="0.014889" ixy="0.00016" iyz="-0.000113" ixz="5.6e-05"/>
+    <inertia ixx="0.014889" iyy="0.020157" izz="0.025166" ixy="5.6e-05" iyz="0.00016" ixz="-0.000113"/>
   </inertial>
   <visual>
@@ -26,10 +26,10 @@
 <link name="wheel_left_forward_link_1">
   <inertial>
-    <origin xyz="0.0038321243790345877 -8.294581043746807e-07 0.0003539119469892979" rpy="0 0 0"/>
+    <origin xyz="0.013345911946989336 0.03374212437903459 -0.04290282945810435" rpy="0 0 0"/>
     <mass value="0.30797982883853386"/>
-    <inertia ixx="0.000267" iyy="0.000139" izz="0.000139" ixy="0.0" iyz="0.0" ixz="0.0"/>
+    <inertia ixx="0.000139" iyy="0.000267" izz="0.000139" ixy="0.0" iyz="0.0" ixz="0.0"/>
   </inertial>
   <visual>
-    <origin xyz="-0.074905 -0.032003 -0.044995" rpy="0 0 0"/>
+    <origin xyz="-0.032003 -0.044995 -0.074905" rpy="0 0 0"/>
     <geometry>
       <mesh filename="file://$(find rcj2025_description)/meshes/wheel_left_forward_link_1.stl" scale="0.001 0.001 0.001"/>
@@ -38,5 +38,5 @@
   </visual>
   <collision>
-    <origin xyz="-0.074905 -0.032003 -0.044995" rpy="0 0 0"/>
+    <origin xyz="-0.032003 -0.044995 -0.074905" rpy="0 0 0"/>
     <geometry>
       <mesh filename="file://$(find rcj2025_description)/meshes/wheel_left_forward_link_1.stl" scale="0.001 0.001 0.001"/>
@@ -46,10 +46,10 @@
 <link name="wheel_right_forward_link_1">
   <inertial>
-    <origin xyz="-0.0038321243830769514 -3.458642732385997e-06 0.0003437339119924457" rpy="0 0 0"/>
+    <origin xyz="0.01333573391199245 -0.12373212438307696 0.10690454135726762" rpy="0 0 0"/>
     <mass value="0.30797982860031553"/>
-    <inertia ixx="0.000267" iyy="0.000139" izz="0.000139" ixy="-0.0" iyz="-0.0" ixz="-0.0"/>
+    <inertia ixx="0.000139" iyy="0.000267" izz="0.000139" ixy="-0.0" iyz="-0.0" ixz="-0.0"/>
   </inertial>
   <visual>
-    <origin xyz="0.074905 -0.032003 -0.044995" rpy="0 0 0"/>
+    <origin xyz="-0.032003 -0.044995 0.074905" rpy="0 0 0"/>
     <geometry>
       <mesh filename="file://$(find rcj2025_description)/meshes/wheel_right_forward_link_1.stl" scale="0.001 0.001 0.001"/>
@@ -58,5 +58,5 @@
   </visual>
   <collision>
-    <origin xyz="0.074905 -0.032003 -0.044995" rpy="0 0 0"/>
+    <origin xyz="-0.032003 -0.044995 0.074905" rpy="0 0 0"/>
     <geometry>
       <mesh filename="file://$(find rcj2025_description)/meshes/wheel_right_forward_link_1.stl" scale="0.001 0.001 0.001"/>
@@ -66,10 +66,10 @@
 <link name="wheel_right_backward_link_1">
   <inertial>
-    <origin xyz="-0.0038321243783342313 6.041397013302474e-06 -0.00012307261745363868" rpy="0 0 0"/>
+    <origin xyz="-0.07712107261745366 -0.033742124378334216 0.1069140413970133" rpy="0 0 0"/>
     <mass value="0.3079798288624377"/>
-    <inertia ixx="0.000267" iyy="0.000139" izz="0.000139" ixy="-0.0" iyz="-0.0" ixz="0.0"/>
+    <inertia ixx="0.000139" iyy="0.000267" izz="0.000139" ixy="0.0" iyz="-0.0" ixz="-0.0"/>
   </inertial>
   <visual>
-    <origin xyz="0.074905 -0.032003 0.044995" rpy="0 0 0"/>
+    <origin xyz="-0.032003 0.044995 0.074905" rpy="0 0 0"/>
     <geometry>
       <mesh filename="file://$(find rcj2025_description)/meshes/wheel_right_backward_link_1.stl" scale="0.001 0.001 0.001"/>
@@ -78,5 +78,5 @@
   </visual>
   <collision>
-    <origin xyz="0.074905 -0.032003 0.044995" rpy="0 0 0"/>
+    <origin xyz="-0.032003 0.044995 0.074905" rpy="0 0 0"/>
     <geometry>
       <mesh filename="file://$(find rcj2025_description)/meshes/wheel_right_backward_link_1.stl" scale="0.001 0.001 0.001"/>
@@ -86,10 +86,10 @@
 <link name="wheel_left_backward_link_1">
   <inertial>
-    <origin xyz="0.003832124382646254 -3.945927425814955e-06 -0.0003437082381777881" rpy="0 0 0"/>
+    <origin xyz="-0.07734170823817779 0.12373212438264627 -0.04290594592742581" rpy="0 0 0"/>
     <mass value="0.30797982861500756"/>
-    <inertia ixx="0.000267" iyy="0.000139" izz="0.000139" ixy="0.0" iyz="0.0" ixz="-0.0"/>
+    <inertia ixx="0.000139" iyy="0.000267" izz="0.000139" ixy="-0.0" iyz="0.0" ixz="0.0"/>
   </inertial>
   <visual>
-    <origin xyz="-0.074905 -0.032003 0.044995" rpy="0 0 0"/>
+    <origin xyz="-0.032003 0.044995 -0.074905" rpy="0 0 0"/>
     <geometry>
       <mesh filename="file://$(find rcj2025_description)/meshes/wheel_left_backward_link_1.stl" scale="0.001 0.001 0.001"/>
@@ -98,5 +98,5 @@
   </visual>
   <collision>
-    <origin xyz="-0.074905 -0.032003 0.044995" rpy="0 0 0"/>
+    <origin xyz="-0.032003 0.044995 -0.074905" rpy="0 0 0"/>
     <geometry>
       <mesh filename="file://$(find rcj2025_description)/meshes/wheel_left_backward_link_1.stl" scale="0.001 0.001 0.001"/>
@@ -105,26 +105,26 @@
 </link>
 <joint name="wheel_left_forward_joint" type="continuous">
-  <origin xyz="0.074905 0.032003 0.044995" rpy="0 0 0"/>
+  <origin xyz="0.032003 0.044995 0.074905" rpy="0 0 0"/>
   <parent link="base_link"/>
   <child link="wheel_left_forward_link_1"/>
-  <axis xyz="1.0 -0.0 -0.0"/>
+  <axis xyz="-0.0 1.0 -0.0"/>
 </joint>
 <joint name="wheel_right_forward_joint" type="continuous">
-  <origin xyz="-0.074905 0.032003 0.044995" rpy="0 0 0"/>
+  <origin xyz="0.032003 0.044995 -0.074905" rpy="0 0 0"/>
   <parent link="base_link"/>
   <child link="wheel_right_forward_link_1"/>
-  <axis xyz="1.0 0.0 0.0"/>
+  <axis xyz="0.0 1.0 0.0"/>
 </joint>
 <joint name="wheel_right_backward_joint" type="continuous">
-  <origin xyz="-0.074905 0.032003 -0.044995" rpy="0 0 0"/>
+  <origin xyz="0.032003 -0.044995 -0.074905" rpy="0 0 0"/>
   <parent link="base_link"/>
   <child link="wheel_right_backward_link_1"/>
-  <axis xyz="-1.0 -0.0 0.0"/>
+  <axis xyz="0.0 -1.0 -0.0"/>
 </joint>
 <joint name="wheel_left_backward_joint" type="continuous">
-  <origin xyz="0.074905 0.032003 -0.044995" rpy="0 0 0"/>
+  <origin xyz="0.032003 -0.044995 0.074905" rpy="0 0 0"/>
   <parent link="base_link"/>
   <child link="wheel_left_backward_link_1"/>
-  <axis xyz="-1.0 0.0 -0.0"/>
+  <axis xyz="-0.0 -1.0 0.0"/>
 </joint>
 </robot>

Commit message: fix: 座標系を修正

File: rcj2025_description/urdf/rcj2025.xacro (robot description, xacro)
@@ -11,5 +11,5 @@
   </inertial>
   <visual>
-    <origin xyz="0 0 0" rpy="0 0 0"/>
+    <origin xyz="0 0 0" rpy="1.57 0 1.57"/>
     <geometry>
       <mesh filename="file://$(find rcj2025_description)/meshes/base_link.stl" scale="0.001 0.001 0.001"/>
@@ -18,5 +18,5 @@
   </visual>
   <collision>
-    <origin xyz="0 0 0" rpy="0 0 0"/>
+    <origin xyz="0 0 0" rpy="1.57 0 1.57"/>
     <geometry>
       <mesh filename="file://$(find rcj2025_description)/meshes/base_link.stl" scale="0.001 0.001 0.001"/>
@@ -31,5 +31,5 @@
   </inertial>
   <visual>
-    <origin xyz="-0.032003 -0.044995 -0.074905" rpy="0 0 0"/>
+    <origin xyz="-0.032003 -0.044995 -0.074905" rpy="1.57 0 1.57"/>
     <geometry>
       <mesh filename="file://$(find rcj2025_description)/meshes/wheel_left_forward_link_1.stl" scale="0.001 0.001 0.001"/>
@@ -38,5 +38,5 @@
   </visual>
   <collision>
-    <origin xyz="-0.032003 -0.044995 -0.074905" rpy="0 0 0"/>
+    <origin xyz="-0.032003 -0.044995 -0.074905" rpy="1.57 0 1.57"/>
     <geometry>
       <mesh filename="file://$(find rcj2025_description)/meshes/wheel_left_forward_link_1.stl" scale="0.001 0.001 0.001"/>
@@ -51,5 +51,5 @@
   </inertial>
   <visual>
-    <origin xyz="-0.032003 -0.044995 0.074905" rpy="0 0 0"/>
+    <origin xyz="-0.032003 -0.044995 0.074905" rpy="1.57 0 1.57"/>
     <geometry>
       <mesh filename="file://$(find rcj2025_description)/meshes/wheel_right_forward_link_1.stl" scale="0.001 0.001 0.001"/>
@@ -58,5 +58,5 @@
   </visual>
   <collision>
-    <origin xyz="-0.032003 -0.044995 0.074905" rpy="0 0 0"/>
+    <origin xyz="-0.032003 -0.044995 0.074905" rpy="1.57 0 1.57"/>
     <geometry>
       <mesh filename="file://$(find rcj2025_description)/meshes/wheel_right_forward_link_1.stl" scale="0.001 0.001 0.001"/>
@@ -71,5 +71,5 @@
   </inertial>
   <visual>
-    <origin xyz="-0.032003 0.044995 0.074905" rpy="0 0 0"/>
+    <origin xyz="-0.032003 0.044995 0.074905" rpy="1.57 0 1.57"/>
     <geometry>
       <mesh filename="file://$(find rcj2025_description)/meshes/wheel_right_backward_link_1.stl" scale="0.001 0.001 0.001"/>
@@ -78,5 +78,5 @@
   </visual>
   <collision>
-    <origin xyz="-0.032003 0.044995 0.074905" rpy="0 0 0"/>
+    <origin xyz="-0.032003 0.044995 0.074905" rpy="1.57 0 1.57"/>
     <geometry>
       <mesh filename="file://$(find rcj2025_description)/meshes/wheel_right_backward_link_1.stl" scale="0.001 0.001 0.001"/>
@@ -91,5 +91,5 @@
   </inertial>
   <visual>
-    <origin xyz="-0.032003 0.044995 -0.074905" rpy="0 0 0"/>
+    <origin xyz="-0.032003 0.044995 -0.074905" rpy="1.57 0 1.57"/>
     <geometry>
       <mesh filename="file://$(find rcj2025_description)/meshes/wheel_left_backward_link_1.stl" scale="0.001 0.001 0.001"/>
@@ -98,5 +98,5 @@
   </visual>
   <collision>
-    <origin xyz="-0.032003 0.044995 -0.074905" rpy="0 0 0"/>
+    <origin xyz="-0.032003 0.044995 -0.074905" rpy="1.57 0 1.57"/>
     <geometry>
       <mesh filename="file://$(find rcj2025_description)/meshes/wheel_left_backward_link_1.stl" scale="0.001 0.001 0.001"/>
@@ -108,5 +108,5 @@
   <parent link="base_link"/>
   <child link="wheel_left_forward_link_1"/>
-  <axis xyz="-0.0 1.0 -0.0"/>
+  <axis xyz="0.0 0.0 1.0"/>
 </joint>
 <joint name="wheel_right_forward_joint" type="continuous">
@@ -114,5 +114,5 @@
   <parent link="base_link"/>
   <child link="wheel_right_forward_link_1"/>
-  <axis xyz="0.0 1.0 0.0"/>
+  <axis xyz="0.0 0.0 1.0"/>
 </joint>
 <joint name="wheel_right_backward_joint" type="continuous">
@@ -120,5 +120,5 @@
   <parent link="base_link"/>
   <child link="wheel_right_backward_link_1"/>
-  <axis xyz="0.0 -1.0 -0.0"/>
+  <axis xyz="0.0 0.0 1.0"/>
 </joint>
 <joint name="wheel_left_backward_joint" type="continuous">
@@ -126,5 +126,5 @@
   <parent link="base_link"/>
   <child link="wheel_left_backward_link_1"/>
-  <axis xyz="-0.0 -1.0 0.0"/>
+  <axis xyz="0.0 0.0 1.0"/>
 </joint>
 </robot>

Commit message: fix: 旋回できない不具合を修正

File: rcj2025_description/urdf/rcj2025.xacro (robot description, xacro)
@@ -11,5 +11,5 @@
   </inertial>
   <visual>
-    <origin xyz="0 0 0" rpy="1.57 0 1.57"/>
+    <origin xyz="0 0 0" rpy="0 0 0"/>
     <geometry>
       <mesh filename="file://$(find rcj2025_description)/meshes/base_link.stl" scale="0.001 0.001 0.001"/>
@@ -18,5 +18,5 @@
   </visual>
   <collision>
-    <origin xyz="0 0 0" rpy="1.57 0 1.57"/>
+    <origin xyz="0 0 0" rpy="0 0 0"/>
     <geometry>
       <mesh filename="file://$(find rcj2025_description)/meshes/base_link.stl" scale="0.001 0.001 0.001"/>
@@ -31,5 +31,5 @@
   </inertial>
   <visual>
-    <origin xyz="-0.032003 -0.044995 -0.074905" rpy="1.57 0 1.57"/>
+    <origin xyz="-0.044995 -0.074905 -0.032003" rpy="0 0 0"/>
     <geometry>
       <mesh filename="file://$(find rcj2025_description)/meshes/wheel_left_forward_link_1.stl" scale="0.001 0.001 0.001"/>
@@ -38,5 +38,5 @@
   </visual>
   <collision>
-    <origin xyz="-0.032003 -0.044995 -0.074905" rpy="1.57 0 1.57"/>
+    <origin xyz="-0.044995 -0.074905 -0.032003" rpy="0 0 0"/>
     <geometry>
       <mesh filename="file://$(find rcj2025_description)/meshes/wheel_left_forward_link_1.stl" scale="0.001 0.001 0.001"/>
@@ -51,5 +51,5 @@
   </inertial>
   <visual>
-    <origin xyz="-0.032003 -0.044995 0.074905" rpy="1.57 0 1.57"/>
+    <origin xyz="-0.044995 0.074905 -0.032003" rpy="0 0 0"/>
     <geometry>
       <mesh filename="file://$(find rcj2025_description)/meshes/wheel_right_forward_link_1.stl" scale="0.001 0.001 0.001"/>
@@ -58,5 +58,5 @@
   </visual>
   <collision>
-    <origin xyz="-0.032003 -0.044995 0.074905" rpy="1.57 0 1.57"/>
+    <origin xyz="-0.044995 0.074905 -0.032003" rpy="0 0 0"/>
     <geometry>
       <mesh filename="file://$(find rcj2025_description)/meshes/wheel_right_forward_link_1.stl" scale="0.001 0.001 0.001"/>
@@ -71,5 +71,5 @@
   </inertial>
   <visual>
-    <origin xyz="-0.032003 0.044995 0.074905" rpy="1.57 0 1.57"/>
+    <origin xyz="0.044995 0.074905 -0.032003" rpy="0 0 0"/>
     <geometry>
       <mesh filename="file://$(find rcj2025_description)/meshes/wheel_right_backward_link_1.stl" scale="0.001 0.001 0.001"/>
@@ -78,5 +78,5 @@
   </visual>
   <collision>
-    <origin xyz="-0.032003 0.044995 0.074905" rpy="1.57 0 1.57"/>
+    <origin xyz="0.044995 0.074905 -0.032003" rpy="0 0 0"/>
     <geometry>
       <mesh filename="file://$(find rcj2025_description)/meshes/wheel_right_backward_link_1.stl" scale="0.001 0.001 0.001"/>
@@ -91,5 +91,5 @@
   </inertial>
   <visual>
-    <origin xyz="-0.032003 0.044995 -0.074905" rpy="1.57 0 1.57"/>
+    <origin xyz="0.044995 -0.074905 -0.032003" rpy="0 0 0"/>
     <geometry>
       <mesh filename="file://$(find rcj2025_description)/meshes/wheel_left_backward_link_1.stl" scale="0.001 0.001 0.001"/>
@@ -98,5 +98,5 @@
   </visual>
   <collision>
-    <origin xyz="-0.032003 0.044995 -0.074905" rpy="1.57 0 1.57"/>
+    <origin xyz="0.044995 -0.074905 -0.032003" rpy="0 0 0"/>
     <geometry>
       <mesh filename="file://$(find rcj2025_description)/meshes/wheel_left_backward_link_1.stl" scale="0.001 0.001 0.001"/>
@@ -105,26 +105,26 @@
 </link>
 <joint name="wheel_left_forward_joint" type="continuous">
-  <origin xyz="0.032003 0.044995 0.074905" rpy="0 0 0"/>
+  <origin xyz="0.044995 0.074905 0.032003" rpy="0 0 0"/>
   <parent link="base_link"/>
   <child link="wheel_left_forward_link_1"/>
-  <axis xyz="0.0 0.0 1.0"/>
+  <axis xyz="0.0 1.0 0.0"/>
 </joint>
 <joint name="wheel_right_forward_joint" type="continuous">
-  <origin xyz="0.032003 0.044995 -0.074905" rpy="0 0 0"/>
+  <origin xyz="0.044995 -0.074905 0.032003" rpy="0 0 0"/>
   <parent link="base_link"/>
   <child link="wheel_right_forward_link_1"/>
-  <axis xyz="0.0 0.0 1.0"/>
+  <axis xyz="0.0 1.0 0.0"/>
 </joint>
 <joint name="wheel_right_backward_joint" type="continuous">
-  <origin xyz="0.032003 -0.044995 -0.074905" rpy="0 0 0"/>
+  <origin xyz="-0.044995 -0.074905 0.032003" rpy="0 0 0"/>
   <parent link="base_link"/>
   <child link="wheel_right_backward_link_1"/>
-  <axis xyz="0.0 0.0 1.0"/>
+  <axis xyz="0.0 1.0 0.0"/>
 </joint>
 <joint name="wheel_left_backward_joint" type="continuous">
-  <origin xyz="0.032003 -0.044995 0.074905" rpy="0 0 0"/>
+  <origin xyz="-0.044995 0.074905 0.032003" rpy="0 0 0"/>
   <parent link="base_link"/>
   <child link="wheel_left_backward_link_1"/>
-  <axis xyz="0.0 0.0 1.0"/>
+  <axis xyz="0.0 1.0 0.0"/>
 </joint>
 </robot>
