Commit message: nav2導入

File: rcj2025_description/urdf/rcj2025.xacro (robot description, xacro)
@@ -128,3 +128,27 @@
   <axis xyz="0.0 1.0 0.0"/>
 </joint>
+<link name="imu_link">
+  <inertial>
+    <mass value="0.01"/>
+    <origin xyz="0 0 0" rpy="0 0 0"/>
+    <inertia ixx="1e-6" ixy="0" ixz="0" iyy="1e-6" iyz="0" izz="1e-6"/>
+  </inertial>
+</link>
+<joint name="imu_joint" type="fixed">
+    <parent link="base_link"/>
+    <child link="imu_link"/>
+    <origin xyz="-0.05 0 0.08" rpy="0 0 0"/>
+</joint>
+<link name="lidar_link">
+    <inertial>
+        <origin xyz="0 0 4" rpy="0 0 0"/>
+        <mass value="0.1"/>
+        <inertia ixx="1e-6" ixy="0" ixz="0" iyy="1e-6" iyz="0" izz="1e-6"/>
+    </inertial>
+</link>
+<joint name="lidar_joint" type="fixed">
+    <parent link="base_link"/>
+    <child link="lidar_link"/>
+    <origin xyz="0.055 0 0.13" rpy="0 0 0"/>
+</joint>
 </robot>

Commit message: feat: nav2動いた

File: rcj2025_description/urdf/rcj2025.xacro (robot description, xacro)
@@ -4,4 +4,10 @@
 <xacro:include filename="$(find rcj2025_description)/urdf/rcj2025.trans" />
 <xacro:include filename="$(find rcj2025_description)/urdf/rcj2025.gazebo" />
+<link name="base_footprint"/>
+<joint name="base_link_joint" type="fixed">
+  <parent link="base_footprint"/>
+  <child link="base_link"/>
+  <origin xyz="0 0 0.009" rpy="0 0 0"/>
+ </joint>
 <link name="base_link">
   <inertial>
@@ -140,5 +146,5 @@
     <origin xyz="-0.05 0 0.08" rpy="0 0 0"/>
 </joint>
-<link name="lidar_link">
+<link name="base_scan">
     <inertial>
         <origin xyz="0 0 4" rpy="0 0 0"/>
@@ -149,5 +155,5 @@
 <joint name="lidar_joint" type="fixed">
     <parent link="base_link"/>
-    <child link="lidar_link"/>
+    <child link="base_scan"/>
     <origin xyz="0.055 0 0.13" rpy="0 0 0"/>
 </joint>
